Commit message: Update robot.urdf

File: robot/robot.urdf (robot description, URDF)
Before this commit: robot ur5_robot, 11 links, 10 joints
Links:
- link base_link_inertia: geometry visual mesh filename=meshes/visual/base.dae
- link forearm_link: geometry visual mesh filename=meshes/visual/forearm.dae
- link shoulder_link: geometry visual mesh filename=meshes/visual/shoulder.dae
- link upper_arm_link: geometry visual mesh filename=meshes/visual/upperarm.dae
- link wrist_1_link: geometry visual mesh filename=meshes/visual/wrist1.dae
- link wrist_2_link: geometry visual mesh filename=meshes/visual/wrist2.dae
- link wrist_3_link: geometry visual mesh filename=meshes/visual/wrist3.dae
